Commit message: robot description udpated

File: src/description/indy_bot_description.urdf (robot description, URDF)
Before this commit: robot indy_bot, 3 links, 2 joints
Links:
- removed link camera_link
- link base_link: geometry 
Joints:
- removed joint camera_joint
- joint lidar_joint: child base_link -> lidar_link; origin xyz=0.0 0.0 ${-(base_height/2+lidar_height/2)} rpy=0 0 0 -> xyz=0.0 0.0 ${(base_height/2+lidar_height/2)} rpy=0 0 0; parent lidar_link -> base_link

Commit message: indy bot model added

File: src/description/indy_bot_description.urdf (robot description, URDF)
Before this commit: robot indy_bot, 2 links, 1 joints
Links:
- removed link lidar_link
- added link camera_link
- added link center_lidar; visual mesh filename=package://indy_bot_urdf/meshes/livox_horizon.stl scale=0.001 0.001 0.001
- added link left_lidar; visual mesh filename=package://indy_bot_urdf/meshes/livox_horizon.stl scale=0.001 0.001 0.001
- added link right_lidar; visual mesh filename=package://indy_bot_urdf/meshes/livox_horizon.stl scale=0.001 0.001 0.001
- link base_link: geometry visual box size=${base_length} ${base_width} ${base_height}
Joints:
- removed joint lidar_joint
- added joint center_lidar_joint: type fixed, parent base_link, child center_lidar, origin xyz=${front_lidar_forward_offset} 0.0 ${(base_height/2+lidar_height/2)} rpy=0 0 0
- added joint left_lidar_joint: type fixed, parent base_link, child left_lidar, origin xyz=0.0 ${side_lidar_offset} ${(base_height/2+lidar_height/2)} rpy=0 0 1.047
- added joint right_lidar_joint: type fixed, parent base_link, child right_lidar, origin xyz=0.0 ${-side_lidar_offset} ${(base_height/2+lidar_height/2)} rpy=0 0 -1.047
- added joint zed_joint: type fixed, parent center_lidar, child camera_link, origin xyz=0.0 0.0 ${lidar_height/2+zed_height/2} rpy=0 0 0

Commit message: berkeley gokart model added

File: src/description/indy_bot_description.urdf (robot description, URDF)
Before this commit: robot indy_bot, 5 links, 4 joints
Links:
- added link chassis; visual box size=${base_length} ${base_width} ${base_height}
- added link sensor_base
- link base_link: geometry 
- link center_lidar: geometry visual mesh filename=package://roar-gokart-urdf/meshes/livox_horizon.stl scale=0.001 0.001 0.001
- link left_lidar: geometry visual mesh filename=package://roar-gokart-urdf/meshes/livox_horizon.stl scale=0.001 0.001 0.001
- link right_lidar: geometry visual mesh filename=package://roar-gokart-urdf/meshes/livox_horizon.stl scale=0.001 0.001 0.001
Joints:
- added joint base_link_to_chassis: type fixed, parent base_link, child chassis, origin xyz=${wheel_base} 0.0 0.0 rpy=0 0 0.0
- added joint sensor_to_chassis: type fixed, parent chassis, child sensor_base, origin xyz=0.0 0.0 ${sensor_base_height} rpy=0 0 0.0
- joint center_lidar_joint: parent base_link -> sensor_base
- joint left_lidar_joint: parent base_link -> sensor_base
- joint right_lidar_joint: parent base_link -> sensor_base
